Commit message: Labortag-Tests, Bug-Fixes, Fehler-Dokumentation

File: bc/data/lara5_candidate.urdf (robot description, URDF)
Before this commit: robot elfin5, 11 links, 10 joints
Joints:
- joint elfin_end_joint: origin xyz=0 -0.0735 0 rpy=1.57079632679 1.57079632679 0 -> xyz=0 -0.059 0 rpy=1.57079632679 1.57079632679 0
- joint elfin_joint2: axis -1 0 0 -> 1 0 0
